File: kicad/rpirfid.sch (KiCad schematic (older format))
At the start: 14 parts

Commit message: added voltage regulator and antenna to schematic
Parts:
- added C? (x3): 10nF, symbol C
- added C? (x4): 100nF, symbol C
- added C? (x2): 1nF, symbol C
- added D? (x4): LED, symbol LED
- added P?: BATTERY INPUT, symbol CONN_01X02
- added R?: R, symbol R
- added R? (x2): 470, symbol R
- added R? (x2): 1k, symbol R
- added U?: EM4095, symbol EM4095
- added U?: LM7805, symbol LM7805
- added U?: LD1117S33CTR, SOT-223, symbol LD1117S33CTR
Connections:
- net labels added: 3.3V, ANT, CDV, EXT_VDD, RES_LED, RFID_CLK, RFID_DATA, RFID_EN, RFID_MOD, RXLED, TXLED, VBATT
- wire segments 42 -> 83
Other:
- note added: "3V REG"
- note added: "5V REG\n"
- note added: "AVR Programmer"
- note added: "BATTERY POWER"
- note added: "POWER LED"
- note added: "Real Time Clock\n"
- note added: "Response LED"
- note added: "TX & RX LED\n"
- note added: "Transceiver/Antenna Circuit"
- note added: "USB INPUT"

Commit message: Trying to add in SD Card & SD Card Datasheet
Parts:
- added 1K: R, symbol R
- added ACT: LED, symbol LED
- added IC1: 4050, symbol 4050
- added IC2: SD_Card_Revised, symbol SD_Card_Revised
Connections:
- net labels added: CD, CLK, CS, DO
- wire segments 83 -> 93

Commit message: SD Card added to the main file
Connections:
- net labels added: DI
- wire segments 93 -> 97
Changed lines of the file:
@@
 LIBS:ds1307
 LIBS:em4095
+LIBS:rpirfid-cache
 EELAYER 25 0
 EELAYER END
@@
 L 4050 IC1
 U 1 1 564FB0B8
-P 3100 6700
-F 0 "IC1" H 3295 6815 60  0000 C CNN
-F 1 "4050" H 3290 6575 60  0000 C CNN
-F 2 "" H 3100 6700 60  0000 C CNN
-F 3 "" H 3100 6700 60  0000 C CNN
-	1    3100 6700
-	1    0    0    -1
-$EndComp
-$Comp
-L 4050 IC1
-U 2 1 564FB161
-P 6000 6450
-F 0 "IC1" H 6195 6565 60  0000 C CNN
-F 1 "4050" H 6190 6325 60  0000 C CNN
-F 2 "" H 6000 6450 60  0000 C CNN
-F 3 "" H 6000 6450 60  0000 C CNN
-	2    6000 6450
-	-1   0    0    1
+P 3100 7050
+F 0 "IC1" H 3295 7165 60  0000 C CNN
+F 1 "4050" H 3290 6925 60  0000 C CNN
+F 2 "" H 3100 7050 60  0000 C CNN
+F 3 "" H 3100 7050 60  0000 C CNN
+	1    3100 7050
+	1    0    0    -1
 $EndComp
 $Comp
 L 4050 IC1
 U 3 1 564FB26D
-P 3100 7350
-F 0 "IC1" H 3295 7465 60  0000 C CNN
-F 1 "4050" H 3290 7225 60  0000 C CNN
-F 2 "" H 3100 7350 60  0000 C CNN
-F 3 "" H 3100 7350 60  0000 C CNN
-	3    3100 7350
+P 2950 5800
+F 0 "IC1" H 3145 5915 60  0000 C CNN
+F 1 "4050" H 3140 5675 60  0000 C CNN
+F 2 "" H 2950 5800 60  0000 C CNN
+F 3 "" H 2950 5800 60  0000 C CNN
+	3    2950 5800
 	1    0    0    -1
 $EndComp
@@
 L 4050 IC1
 U 4 1 564FB302
-P 1800 7200
-F 0 "IC1" H 1995 7315 60  0000 C CNN
-F 1 "4050" H 1990 7075 60  0000 C CNN
-F 2 "" H 1800 7200 60  0000 C CNN
-F 3 "" H 1800 7200 60  0000 C CNN
-	4    1800 7200
-	0    1    1    0
+P 1800 6150
+F 0 "IC1" H 1995 6265 60  0000 C CNN
+F 1 "4050" H 1990 6025 60  0000 C CNN
+F 2 "" H 1800 6150 60  0000 C CNN
+F 3 "" H 1800 6150 60  0000 C CNN
+	4    1800 6150
+	1    0    0    -1
 $EndComp
 $Comp
 L 4050 IC1
 U 5 1 564FB3C5
-P 5300 5600
-F 0 "IC1" H 5495 5715 60  0000 C CNN
-F 1 "4050" H 5490 5475 60  0000 C CNN
-F 2 "" H 5300 5600 60  0000 C CNN
-F 3 "" H 5300 5600 60  0000 C CNN
-	5    5300 5600
+P 2750 7400
+F 0 "IC1" H 2945 7515 60  0000 C CNN
+F 1 "4050" H 2940 7275 60  0000 C CNN
+F 2 "" H 2750 7400 60  0000 C CNN
+F 3 "" H 2750 7400 60  0000 C CNN
+	5    2750 7400
 	1    0    0    -1
 $EndComp
@@
 L 4050 IC1
 U 6 1 564FB472
-P 3600 5750
-F 0 "IC1" H 3795 5865 60  0000 C CNN
-F 1 "4050" H 3790 5625 60  0000 C CNN
-F 2 "" H 3600 5750 60  0000 C CNN
-F 3 "" H 3600 5750 60  0000 C CNN
-	6    3600 5750
+P 4850 7450
+F 0 "IC1" H 5045 7565 60  0000 C CNN
+F 1 "4050" H 5040 7325 60  0000 C CNN
+F 2 "" H 4850 7450 60  0000 C CNN
+F 3 "" H 4850 7450 60  0000 C CNN
+	6    4850 7450
 	1    0    0    -1
 $EndComp
@@
 Connection ~ 6900 5000
 Wire Wire Line
-	5550 6450 5200 6450
-Wire Wire Line
-	3850 6700 3550 6700
-Wire Wire Line
-	1250 6700 2650 6700
+	600  7050 2650 7050
 $Comp
 L GND #PWR?
 U 1 1 56500BC2
-P 2900 5850
-F 0 "#PWR?" H 2900 5600 50  0001 C CNN
-F 1 "GND" H 2900 5700 50  0000 C CNN
-F 2 "" H 2900 5850 60  0000 C CNN
-F 3 "" H 2900 5850 60  0000 C CNN
-	1    2900 5850
-	1    0    0    -1
-$EndComp
-Wire Wire Line
-	3150 5750 2900 5750
-Wire Wire Line
-	2900 5750 2900 5850
-Wire Wire Line
-	4550 5600 4850 5600
-Text Label 1250 6700 0    60   ~ 0
+P 3900 7450
+F 0 "#PWR?" H 3900 7200 50  0001 C CNN
+F 1 "GND" H 3900 7300 50  0000 C CNN
+F 2 "" H 3900 7450 60  0000 C CNN
+F 3 "" H 3900 7450 60  0000 C CNN
+	1    3900 7450
+	0    1    1    0
+$EndComp
+Wire Wire Line
+	3900 7450 4400 7450
+Text Label 600  7050 0    60   ~ 0
 CLK
 $Comp
@@
 L GND #PWR?
 U 1 1 56504438
-P 4550 5700
-F 0 "#PWR?" H 4550 5450 50  0001 C CNN
-F 1 "GND" H 4550 5550 50  0000 C CNN
-F 2 "" H 4550 5700 60  0000 C CNN
-F 3 "" H 4550 5700 60  0000 C CNN
-	1    4550 5700
-	1    0    0    -1
-$EndComp
-Wire Wire Line
-	4550 5700 4550 5600
+P 1800 7500
+F 0 "#PWR?" H 1800 7250 50  0001 C CNN
+F 1 "GND" H 1800 7350 50  0000 C CNN
+F 2 "" H 1800 7500 60  0000 C CNN
+F 3 "" H 1800 7500 60  0000 C CNN
+	1    1800 7500
+	1    0    0    -1
+$EndComp
 Wire Wire Line
 	6650 6450 6450 6450
@@
 L R 1K
 U 1 1 56506416
-P 3400 7700
-F 0 "1K " V 3480 7700 50  0000 C CNN
-F 1 "R" V 3400 7700 50  0000 C CNN
-F 2 "" V 3330 7700 30  0000 C CNN
-F 3 "" H 3400 7700 30  0000 C CNN
-	1    3400 7700
+P 3150 6150
+F 0 "1K " V 3230 6150 50  0000 C CNN
+F 1 "R" V 3150 6150 50  0000 C CNN
+F 2 "" V 3080 6150 30  0000 C CNN
+F 3 "" H 3150 6150 30  0000 C CNN
+	1    3150 6150
 	0    1    1    0
 $EndComp
@@
 L LED ACT
 U 1 1 56506507
-P 2800 7700
-F 0 "ACT RED" H 2800 7800 50  0000 C CNN
-F 1 "LED" H 2800 7600 50  0000 C CNN
-F 2 "" H 2800 7700 60  0000 C CNN
-F 3 "" H 2800 7700 60  0000 C CNN
-	1    2800 7700
+P 2650 6150
+F 0 "ACT RED" H 2650 6250 50  0000 C CNN
+F 1 "LED" H 2650 6050 50  0000 C CNN
+F 2 "" H 2650 6150 60  0000 C CNN
+F 3 "" H 2650 6150 60  0000 C CNN
+	1    2650 6150
 	-1   0    0    1
 $EndComp
 Wire Wire Line
-	1800 6750 1800 6700
-Connection ~ 1800 6700
-Wire Wire Line
-	1800 7650 1800 7700
-Wire Wire Line
-	1800 7700 2600 7700
-Wire Wire Line
-	3000 7700 3250 7700
-Wire Wire Line
-	3900 7100 3900 7700
-Wire Wire Line
-	3900 7700 3550 7700
-Wire Wire Line
-	3550 7350 3900 7350
-Connection ~ 3900 7350
-Wire Wire Line
-	2350 7350 2650 7350
-Text Label 2200 7350 0    60   ~ 0
+	2100 5800 2500 5800
+Text Label 2100 5800 0    60   ~ 0
 CS
-Wire Wire Line
-	3100 6300 3100 6550
-Wire Wire Line
-	3100 6550 3850 6550
-Text Label 3100 6300 0    60   ~ 0
+Text Label 1750 6850 0    60   ~ 0
 3.3V
 Text Label 6050 6000 0    60   ~ 0
 DO
 Wire Wire Line
-	6050 6000 6050 6250
-Wire Wire Line
-	6050 6250 5500 6250
-Wire Wire Line
-	5500 6250 5500 6300
-Wire Wire Line
-	5500 6300 5200 6300
+	6050 6300 6050 6000
+Wire Wire Line
+	5200 6300 6050 6300
+Text Label 6650 6450 0    60   ~ 0
+DI
+Wire Wire Line
+	3850 6700 3750 6700
+Wire Wire Line
+	3750 6700 3750 7050
+Wire Wire Line
+	3750 7050 3550 7050
+Wire Wire Line
+	2250 6150 2450 6150
+Wire Wire Line
+	2850 6150 3000 6150
+Wire Wire Line
+	3400 5800 3550 5800
+Wire Wire Line
+	3550 5800 3550 6250
+Connection ~ 3550 6150
+Wire Wire Line
+	1350 6150 1250 6150
+Wire Wire Line
+	1250 6150 1250 7050
+Connection ~ 1250 7050
+$Comp
+L 4050 IC1
+U 2 1 564FB161
+P 2200 6500
+F 0 "IC1" H 2395 6615 60  0000 C CNN
+F 1 "4050" H 2390 6375 60  0000 C CNN
+F 2 "" H 2200 6500 60  0000 C CNN
+F 3 "" H 2200 6500 60  0000 C CNN
+	2    2200 6500
+	1    0    0    -1
+$EndComp
+Wire Wire Line
+	3850 6550 2800 6550
+Wire Wire Line
+	2800 6550 2800 6850
+Wire Wire Line
+	2800 6850 1750 6850
+Wire Wire Line
+	3850 6400 2800 6400
+Wire Wire Line
+	2800 6400 2800 6500
+Wire Wire Line
+	2800 6500 2650 6500
+Text Label 1500 6500 0    60   ~ 0
+DI
+Wire Wire Line
+	1500 6500 1750 6500
+Wire Wire Line
+	3550 6150 3300 6150
+Wire Wire Line
+	3550 6250 3850 6250
+Wire Wire Line
+	2300 7400 1800 7400
+Wire Wire Line
+	1800 7400 1800 7500
 $EndSCHEMATC

Commit message: Slight update with GND
Connections:
- wire segments 97 -> 98
Changed lines of the file:
@@
 Wire Wire Line
 	1800 7400 1800 7500
+$Comp
+L GND #PWR?
+U 1 1 56525B6E
+P 750 600
+F 0 "#PWR?" H 750 350 50  0001 C CNN
+F 1 "GND" H 750 450 50  0000 C CNN
+F 2 "" H 750 600 60  0000 C CNN
+F 3 "" H 750 600 60  0000 C CNN
+	1    750  600
+	0    1    1    0
+$EndComp
+Text Label 1150 600  0    60   ~ 0
+GND
+Wire Wire Line
+	1150 600  750  600
 $EndSCHEMATC

Commit message: Fixed Labels and Connected SD Card to Microcontroller
Connections:
- net labels removed: AVG_MOSI, AVR_SCK
- wire segments 98 -> 101
Changed lines of the file:
@@
 AVR_MISO
 Text Label 4800 950  2    60   ~ 0
-AVR_SCK
+AVR_SCLK
 Text Label 4800 1050 2    60   ~ 0
 AVR_RESET
@@
 VCC
 Text Label 5300 950  0    60   ~ 0
-AVG_MOSI
+AVR_MOSI
 Text Label 5300 1050 0    60   ~ 0
 GND
@@
 	1    0    0    -1
 $EndComp
-Wire Wire Line
-	6650 6450 6450 6450
 $Comp
 L R 1K
@@
 Wire Wire Line
 	5200 6300 6050 6300
-Text Label 6650 6450 0    60   ~ 0
-DI
 Wire Wire Line
 	3850 6700 3750 6700
@@
 Wire Wire Line
 	1150 600  750  600
+Text Label 4450 5350 0    60   ~ 0
+AVR_MISO
+Text Label 4450 5550 0    60   ~ 0
+AVR_SCLK
+Text Label 5200 5300 0    60   ~ 0
+AVR_MOSI
+Text Label 5200 5550 0    60   ~ 0
+AVR_RESET
+Text Label 4050 5550 0    60   ~ 0
+CLK
+Wire Wire Line
+	4450 5550 4050 5550
+Text Label 5850 5300 0    60   ~ 0
+DI
+Wire Wire Line
+	5850 5300 5200 5300
+Text Label 4100 5350 0    60   ~ 0
+DO
+Wire Wire Line
+	4100 5350 4450 5350
+Text Label 5900 5550 0    60   ~ 0
+CD
+Wire Wire Line
+	5900 5550 5200 5550
 $EndSCHEMATC

Commit message: Fully connected SD Card and labels
Parts:
- IC2: symbol SD_Card_Revised -> SD_Card_Revised-RESCUE-rpirfid
- renumbered 1K to 1K~, ACT to ACT~RED
Connections:
- net labels added: CardDetect, CardSelect, DataInput, DataOutput, SPI_CLK
- net labels removed: CD, CLK, CS, DI, DO
- wire segments 101 -> 100
- no-connect marks 1 -> 6
Changed lines of the file:
@@
 EESchema Schematic File Version 2
+LIBS:rpirfid-rescue
 LIBS:power
 LIBS:device
@@
 3V REG
 $Comp
-L SD_Card_Revised IC2
+L SD_Card_Revised-RESCUE-rpirfid IC2
 U 1 1 564FAFEB
 P 4600 6400
@@
 	3900 7450 4400 7450
 Text Label 600  7050 0    60   ~ 0
-CLK
+SPI_CLK
 $Comp
 L GND #PWR?
@@
 Wire Wire Line
 	5600 6600 5200 6600
-Text Label 5550 6900 0    60   ~ 0
-CD
+Text Label 5600 6800 0    60   ~ 0
+CardDetect
 $Comp
 L GND #PWR?
@@
 $EndComp
 $Comp
-L R 1K
+L R 1K~
 U 1 1 56506416
 P 3150 6150
@@
 $EndComp
 $Comp
-L LED ACT
+L LED ACT~RED
 U 1 1 56506507
 P 2650 6150
@@
 $EndComp
 Wire Wire Line
-	2100 5800 2500 5800
-Text Label 2100 5800 0    60   ~ 0
-CS
+	1850 5800 2500 5800
+Text Label 1850 5800 0    60   ~ 0
+CardSelect
 Text Label 1750 6850 0    60   ~ 0
 3.3V
 Text Label 6050 6000 0    60   ~ 0
-DO
+DataOutput
 Wire Wire Line
 	6050 6300 6050 6000
@@
 Connection ~ 3550 6150
 Wire Wire Line
-	1350 6150 1250 6150
-Wire Wire Line
-	1250 6150 1250 7050
-Connection ~ 1250 7050
+	1350 6150 1100 6150
+Wire Wire Line
+	1100 6150 1100 7050
+Connection ~ 1100 7050
 $Comp
 L 4050 IC1
@@
 Wire Wire Line
 	2800 6500 2650 6500
-Text Label 1500 6500 0    60   ~ 0
-DI
-Wire Wire Line
-	1500 6500 1750 6500
+Text Label 1200 6500 0    60   ~ 0
+DataInput
+Wire Wire Line
+	1200 6500 1750 6500
 Wire Wire Line
 	3550 6150 3300 6150
@@
 Wire Wire Line
 	1150 600  750  600
-Text Label 4450 5350 0    60   ~ 0
+Text Label 1250 5300 0    60   ~ 0
 AVR_MISO
-Text Label 4450 5550 0    60   ~ 0
+Text Label 1250 5450 0    60   ~ 0
 AVR_SCLK
-Text Label 5200 5300 0    60   ~ 0
+Text Label 1250 5100 0    60   ~ 0
 AVR_MOSI
-Text Label 5200 5550 0    60   ~ 0
-AVR_RESET
-Text Label 4050 5550 0    60   ~ 0
-CLK
-Wire Wire Line
-	4450 5550 4050 5550
-Text Label 5850 5300 0    60   ~ 0
-DI
-Wire Wire Line
-	5850 5300 5200 5300
-Text Label 4100 5350 0    60   ~ 0
-DO
-Wire Wire Line
-	4100 5350 4450 5350
-Text Label 5900 5550 0    60   ~ 0
-CD
-Wire Wire Line
-	5900 5550 5200 5550
+Text Label 650  5450 0    60   ~ 0
+SPI_CLK
+Wire Wire Line
+	1250 5450 650  5450
+Text Label 650  5100 0    60   ~ 0
+DataInput
+Wire Wire Line
+	650  5100 1250 5100
+Text Label 650  5300 0    60   ~ 0
+DataOutput
+Wire Wire Line
+	650  5300 1250 5300
+Text Label 4950 2700 0    60   ~ 0
+CardSelect
+Text Label 4950 2900 0    60   ~ 0
+CardDetect
+NoConn ~ 5300 7450
+NoConn ~ 3200 7400
+NoConn ~ 5200 6450
+NoConn ~ 3850 6150
+NoConn ~ 5200 6700
 $EndSCHEMATC

Commit message: PCB was started
Parts:
- 1K1: renamed from 1K~; footprint (none) -> Resistors_SMD:R_1210
- ACT1: renamed from ACT~RED; footprint (none) -> LEDs:LED-1206
- C1, C10, C11, C12, C2, C3, C4, C5, C6, C7, C8, C9: renamed from C?; footprint (none) -> Capacitors_SMD:C_1206
- Crystal1: renamed from Crystal; footprint (none) -> Crystals:Crystal_Round_Horizontal_2mm
- D1, D2, D3, D4: renamed from D?; footprint (none) -> LEDs:LED-1206
- IC2: footprint (none) -> Custom_Library:SD_Card
- P1: renamed from P?; footprint (none) -> Connect:USB_A
- P2, P3, P4: renamed from P?; footprint (none) -> Connect:AK300-2
- R1, R2, R3, R4, R5, R6, R7, R8: renamed from R?; footprint (none) -> Resistors_SMD:R_1206
- SW1: renamed from SW?; footprint (none) -> Buttons_Switches_ThroughHole:SW_PUSH_SMALL
- U1: renamed from U?; footprint TQFP44 -> (none)
- U2: renamed from U?; footprint (none) -> ds1308:ds1307
- U5: renamed from U?; footprint SOT-223 -> (none)
- X1: renamed from X?; footprint (none) -> Crystals:Crystal_Round_Vertical_2mm
- gave numbers to parts that had none: 2

Commit message: new stuff
Parts:
- IC1: footprint (none) -> HEX4050:HEX4045
- U1: footprint (none) -> tqfp44:TQFP_44
- U2: symbol ds1307 -> ds1307-RESCUE-rpirfid
- U3: footprint (none) -> Housings_SOIC:SOIC-16_3.9x9.9mm_Pitch1.27mm
- U4: footprint (none) -> Connect:PINHEAD1-3; symbol LM7805 -> LM7805-RESCUE-rpirfid
- U5: footprint (none) -> Connect:PINHEAD1-3
Connections:
- net labels removed: EXT_VDD
Changed lines of the file:
@@
 LIBS:ds1307
 LIBS:em4095
+LIBS:7805
 LIBS:rpirfid-cache
 EELAYER 25 0
@@
 F 0 "U1" H 2900 5250 40  0000 C CNN
 F 1 "ATMEGA32U4-A" H 4550 2050 40  0000 C CNN
-F 2 "" H 3850 3550 35  0001 C CIN
+F 2 "tqfp44:TQFP_44" H 3850 3550 35  0001 C CIN
 F 3 "" H 4950 4650 60  0000 C CNN
 	1    3850 3550
@@
 $EndComp
 $Comp
-L ds1307 U2
+L ds1307-RESCUE-rpirfid U2
 U 1 1 563DECB3
 P 7600 1700
@@
 F 0 "U3" H 7600 3150 60  0000 C CNN
 F 1 "EM4095" H 7600 4300 60  0000 C CNN
-F 2 "" H 7600 3550 60  0001 C CNN
+F 2 "Housings_SOIC:SOIC-16_3.9x9.9mm_Pitch1.27mm" H 7600 3550 60  0001 C CNN
 F 3 "" H 7600 3550 60  0000 C CNN
 	1    7600 3550
@@
 TXLED
 $Comp
-L LM7805 U4
+L LM7805-RESCUE-rpirfid U4
 U 1 1 5652D2E3
 P 8500 5250
 F 0 "U4" H 8650 5054 60  0000 C CNN
 F 1 "LM7805" H 8500 5450 60  0000 C CNN
-F 2 "" H 8500 5250 60  0001 C CNN
+F 2 "Connect:PINHEAD1-3" H 8500 5250 60  0001 C CNN
 F 3 "" H 8500 5250 60  0000 C CNN
 	1    8500 5250
@@
 Text Label 8100 5200 2    60   ~ 0
 VBATT
-Text Label 8900 5200 0    60   ~ 0
-EXT_VDD
 Text Notes 7950 5350 0    60   ~ 0
 5V REG\n
@@
 F 0 "U5" H 9700 6050 40  0000 C CNN
 F 1 "LD1117S33CTR" H 9700 6000 40  0000 C CNN
-F 2 "" H 9700 5900 40  0001 C CNN
+F 2 "Connect:PINHEAD1-3" H 9700 5900 40  0001 C CNN
 F 3 "" H 9700 5800 60  0000 C CNN
 	1    9700 5800
@@
 F 0 "IC1" H 3295 7165 60  0000 C CNN
 F 1 "4050" H 3290 6925 60  0000 C CNN
-F 2 "" H 3100 7050 60  0001 C CNN
+F 2 "HEX4050:HEX4045" H 3100 7050 60  0001 C CNN
 F 3 "" H 3100 7050 60  0000 C CNN
 	1    3100 7050
@@
 F 0 "IC1" H 3145 5915 60  0000 C CNN
 F 1 "4050" H 3140 5675 60  0000 C CNN
-F 2 "" H 2950 5800 60  0001 C CNN
+F 2 "HEX4050:HEX4045" H 2950 5800 60  0001 C CNN
 F 3 "" H 2950 5800 60  0000 C CNN
 	3    2950 5800
@@
 F 0 "IC1" H 1995 6265 60  0000 C CNN
 F 1 "4050" H 1990 6025 60  0000 C CNN
-F 2 "" H 1800 6150 60  0001 C CNN
+F 2 "HEX4050:HEX4045" H 1800 6150 60  0001 C CNN
 F 3 "" H 1800 6150 60  0000 C CNN
 	4    1800 6150
@@
 F 0 "IC1" H 2945 7515 60  0000 C CNN
 F 1 "4050" H 2940 7275 60  0000 C CNN
-F 2 "" H 2750 7400 60  0001 C CNN
+F 2 "HEX4050:HEX4045" H 2750 7400 60  0001 C CNN
 F 3 "" H 2750 7400 60  0000 C CNN
 	5    2750 7400
@@
 F 0 "IC1" H 5045 7565 60  0000 C CNN
 F 1 "4050" H 5040 7325 60  0000 C CNN
-F 2 "" H 4850 7450 60  0001 C CNN
+F 2 "HEX4050:HEX4045" H 4850 7450 60  0001 C CNN
 F 3 "" H 4850 7450 60  0000 C CNN
 	6    4850 7450
@@
 F 0 "IC1" H 2395 6615 60  0000 C CNN
 F 1 "4050" H 2390 6375 60  0000 C CNN
-F 2 "" H 2200 6500 60  0001 C CNN
+F 2 "HEX4050:HEX4045" H 2200 6500 60  0001 C CNN
 F 3 "" H 2200 6500 60  0000 C CNN
 	2    2200 6500
