File: kicad/rpirfid.sch (KiCad schematic (older format))
At the start: 40 parts, among them IC1 4050, IC2 SD_Card_Revised, P1 USB_A, P2 POWER, P3 AVR_PRG_SPI, P4 BATTERY INPUT, SW1 SW_PUSH, U1 ATMEGA32U4-A, U2 ds1307, U3 EM4095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

Commit message: all but sd card associated
Parts:
- removed IC2: SD_Card_Revised, Custom_Library:SD_Card, symbol SD_Card_Revised-RESCUE-rpirfid
- removed U2: ds1307, ds1308:ds1307, symbol ds1307-RESCUE-rpirfid
- added U2: SD_Card_Revised, Housings_DIP:DIP-8_W7.62mm, symbol SD_Card_Revised
- added U6: ds1307, Housings_DIP:DIP-8_W7.62mm, symbol ds1307
Changed lines of the file:
@@
 	0    1    1    0
-$EndComp
-$Comp
-L ds1307-RESCUE-rpirfid U2
-U 1 1 563DECB3
-P 7600 1700
-F 0 "U2" H 7650 2350 60  0000 C CNN
-F 1 "ds1307" H 7600 1750 60  0000 C CNN
-F 2 "ds1308:ds1307" H 8050 1800 60  0001 C CNN
-F 3 "" H 8050 1800 60  0000 C CNN
-	1    7600 1700
-	1    0    0    -1
 $EndComp
 Text Label 8200 1500 0    60   ~ 0
@@
 3V REG
 $Comp
-L SD_Card_Revised-RESCUE-rpirfid IC2
-U 1 1 564FAFEB
-P 4600 6400
-F 0 "IC2" H 4550 6700 60  0000 C CNN
-F 1 "SD_Card_Revised" H 4600 6800 60  0000 C CNN
-F 2 "Custom_Library:SD_Card" H 4700 6400 60  0001 C CNN
-F 3 "" H 4700 6400 60  0000 C CNN
-	1    4600 6400
-	1    0    0    -1
-$EndComp
-$Comp
 L 4050 IC1
 U 1 1 564FB0B8
@@
 NoConn ~ 3850 6150
 NoConn ~ 5200 6700
+$Comp
+L ds1307 U6
+U 1 1 566B2499
+P 7600 1700
+F 0 "U6" H 7650 2350 60  0000 C CNN
+F 1 "ds1307" H 7600 1750 60  0000 C CNN
+F 2 "Housings_DIP:DIP-8_W7.62mm" H 8050 1800 60  0001 C CNN
+F 3 "" H 8050 1800 60  0000 C CNN
+	1    7600 1700
+	1    0    0    -1
+$EndComp
+$Comp
+L SD_Card_Revised U2
+U 1 1 566B51B1
+P 4600 6400
+F 0 "U2" H 4550 6700 60  0000 C CNN
+F 1 "SD_Card_Revised" H 4600 6800 60  0000 C CNN
+F 2 "Housings_DIP:DIP-8_W7.62mm" H 4700 6400 60  0001 C CNN
+F 3 "" H 4700 6400 60  0000 C CNN
+	1    4600 6400
+	1    0    0    -1
+$EndComp
 $EndSCHEMATC
