File: kicad/rpirfid.kicad_pcb (KiCad board)
At the start: 2 copper layers, 0 parts

Commit message: PCB layout
Parts:
- added 1K1: R, Resistors_SMD:R_1210, F.Cu at (99.0, 39.5)
- added ACT1: LED, LEDs:LED-1206, F.Cu at (105.0, 39.5)
- added C1: 1uF, Capacitors_SMD:C_1206, F.Cu at (146.5, 55.2)
- added C10: 100nF, Capacitors_SMD:C_1206, F.Cu at (157.5, 60.7)
- added C11: 100nF, Capacitors_SMD:C_1206, F.Cu at (157.5, 63.8)
- added C12: 1nF, Capacitors_SMD:C_1206, F.Cu at (152.0, 56.8)
- added C2: 1uF, Capacitors_SMD:C_1206, F.Cu at (108.0, 58.2)
- added C3: 1uF, Capacitors_SMD:C_1206, F.Cu at (108.0, 52.5)
- added C4: 100nF, Capacitors_SMD:C_1206, F.Cu at (137.7, 57.1)
- added C5: 10nF, Capacitors_SMD:C_1206, F.Cu at (137.7, 62.7)
- added C6: 10nF, Capacitors_SMD:C_1206, F.Cu at (138.0, 59.8)
- added C7: 10nF, Capacitors_SMD:C_1206, F.Cu at (137.7, 65.7)
- added C8: 1nF, Capacitors_SMD:C_1206, F.Cu at (152.0, 59.8)
- added C9: 100nF, Capacitors_SMD:C_1206, F.Cu at (157.5, 57.7)
- added Crystal1: 32.768kHz, Crystals:Crystal_Round_Horizontal_2mm, F.Cu at (128.2, 75.8)
- added D1: LED, LEDs:LED-1206, F.Cu at (111.5, 69.8)
- added D2: LED, LEDs:LED-1206, F.Cu at (100.0, 70.0)
- added D3: LED, LEDs:LED-1206, F.Cu at (126.5, 70.0)
- added D4: LED, LEDs:LED-1206, F.Cu at (131.5, 59.2)
- added IC1: 4050, HEX4050:HEX4045, F.Cu at (124.0, 40.0)
- added P1: USB_A, Connect:USB_A, F.Cu at (143.5, 35.5)
- added P2: POWER, Connect:AK300-2, F.Cu at (110.0, 79.0)
- added P3: AVR_PRG_SPI, Connect:AK300-2, F.Cu at (99.0, 79.0)
- added P4: BATTERY INPUT, Connect:AK300-2, F.Cu at (151.5, 78.5)
- added R1: 22, Resistors_SMD:R_1206, F.Cu at (149.5, 50.5)
- added R2: 22, Resistors_SMD:R_1206, F.Cu at (144.5, 50.5)
- added R3: 10k, Resistors_SMD:R_1206, F.Cu at (123.0, 83.0)
- added R4: 470, Resistors_SMD:R_1206, F.Cu at (105.0, 70.0)
- added R5: 1k, Resistors_SMD:R_1206, F.Cu at (116.5, 69.8)
- added R6: 1k, Resistors_SMD:R_1206, F.Cu at (128.2, 82.5)
- added R7: 470, Resistors_SMD:R_1206, F.Cu at (131.5, 56.5)
- added R8: R, Resistors_SMD:R_1206, F.Cu at (151.9, 63.2)
- added SW1: SW_PUSH, Buttons_Switches_ThroughHole:SW_PUSH_SMALL, F.Cu at (123.0, 77.0)
- added U1: ATMEGA32U4-A, tqfp44:TQFP_44, F.Cu at (119.8, 58.0)
- added U2: SD_Card_Revised, Housings_DIP:DIP-8_W7.62mm, B.Cu at (106.5, 43.5)
- added U3: EM4095, Housings_SOIC:SOIC-16_3.9x9.9mm_Pitch1.27mm, F.Cu at (145.0, 61.8)
- added U4: LM7805, Connect:PINHEAD1-3, F.Cu at (101.0, 56.0)
- added U5: LD1117S33CTR, Connect:PINHEAD1-3, F.Cu at (101.0, 49.0)
- added U6: ds1307, Housings_DIP:DIP-8_W7.62mm, F.Cu at (131.2, 74.5)
- added X1: CRYSTAL_SMD, Crystals:Crystal_Round_Vertical_2mm, F.Cu at (122.0, 68.0)
Other:
- board outline added: 64 x 51 mm
