File: kicad/_autosave-rpirfid.kicad_pcb (KiCad board)
At the start: 2 copper layers, 64 x 51 mm, 40 parts, among them IC1 4050, P1 USB_A, P2 POWER, P3 AVR_PRG_SPI, P4 BATTERY INPUT, SW1 SW_PUSH, U1 ATMEGA32U4-A, U2 SD_Card_Revised, U3 EM4095, U4 LM7805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

Commit message: Routing
Parts:
- moved R3 3.87 mm to (145.4, 79.6)
Routing:
- net /AVR_RESET: track 59.3 -> 65.4 mm
- net VCC: track 47.5 -> 44.4 mm
- net GND: track 127.7 -> 126.5 mm
